File: kicad_board_files/electro_pet.sch (KiCad schematic (older format))
At the start: 15 parts, among them SW1 SWITCH_INV, SW2 SW_PUSH, SW3 SW_PUSH, U1 8X8_LED_MATRIX, U2 SMALL_LIPO_CHARGER, U3 ELECTRO_HAT, U4 3.3_VOLTAGE_REG, U5 MPU-6050, U6 SMALL_DC_DC_BOOST, U7 ARDUINO_PRO_MICRO, U8 BATTERY_CUSTOM, U9 A3144

Commit message: fixed a wiring issue with the switch
Connections:
- wire segments 79 -> 76
Changed lines of the file:
@@
 Sheet 1 1
 Title ""
-Date "15 sep 2016"
+Date "17 oct 2016"
 Rev ""
 Comp ""
@@
 	4350 2300 4700 2300
 Wire Wire Line
-	4700 2300 4700 2150
-Wire Wire Line
-	4700 2150 5400 2150
-Wire Wire Line
-	5400 2150 5400 3250
-Wire Wire Line
-	5400 3250 4350 3250
-Wire Wire Line
-	2900 2650 3350 2650
+	2900 2650 4350 2650
 Connection ~ 4500 3350
 Connection ~ 4500 2750
@@
 Wire Wire Line
 	3000 6600 3000 6650
+Wire Wire Line
+	4350 2650 4350 3250
+Connection ~ 3350 2650
 $EndSCHEMATC
